Commit message: replace panda.h with generated one

File: models/franka_description/panda.urdf (robot description, URDF)
Before this commit: robot panda, 8 links, 7 joints
Links:
- link panda_link0: geometry collision mesh filename=meshes/Simplified/watertight/link0.obj; visual mesh filename=meshes/Simplified/watertight/link0.obj
- link panda_link1: geometry collision mesh filename=meshes/Simplified/watertight/link1.obj; visual mesh filename=meshes/Simplified/watertight/link1.obj
- link panda_link2: geometry collision mesh filename=meshes/Simplified/watertight/link2.obj; visual mesh filename=meshes/Simplified/watertight/link2.obj
- link panda_link3: geometry collision mesh filename=meshes/Simplified/watertight/link3.obj; visual mesh filename=meshes/Simplified/watertight/link3.obj
- link panda_link4: geometry collision mesh filename=meshes/Simplified/watertight/link4.obj; visual mesh filename=meshes/Simplified/watertight/link4.obj
- link panda_link5: geometry collision mesh filename=meshes/Simplified/watertight/link5.obj; visual mesh filename=meshes/Simplified/watertight/link5.obj
- link panda_link6: geometry collision mesh filename=meshes/Simplified/watertight/link6.obj; visual mesh filename=meshes/Simplified/watertight/link6.obj
- link panda_link7: geometry collision mesh filename=meshes/Simplified/watertight/link7_nohand.obj; visual mesh filename=meshes/Simplified/watertight/link7_nohand.obj
